File: 8-Bit-Computer/8-Bit-Computer.kicad_sch (KiCad schematic)
At the start: 50 parts, among them J1 XLR3_Switched, J2 XLR3_Switched, SW1 SW_Push, SW2 SW_DIP_x04, U1 NA555D, U10 74LS283, U11 74HC245, U12 74HC86, U13 74HC86, U14 74HC245, U15 HM62256BLP, U16 74HC245, U17 74157, U18 74157, U19 74157, U2 AMS1117-5.0, U20 74HC00, U21 74157, U22 74173, U3 74HC00, U4 LM555xM, U5 NA555D, U6 74HC00, U7 74HC245, U8 74HC245, U9 74LS283

Commit message: mem done. will review tomorrow.
Parts:
- removed D2: R_LED, symbol Device:LED
- added C8: C_Small, symbol Device:C_Small
- added D3, D4, D5, D6: G_LED, symbol Device:LED
- added D7: R_LED, symbol Device:LED
- added R13, R14, R15, R16: R_US, symbol Device:R_US
- added R17, R18, R19, R20, R21, R22, R23, R24: 1 Mohm, symbol Device:R_US
- added R25: 10 Kohm, symbol Device:R_US
- added R26: 1 kOhm, symbol Device:R_US
- added SW3: SW_DIP_x08, symbol Switch:SW_DIP_x08
- added SW4: SW_Push, symbol Switch:SW_Push
Connections:
- net +5V: now also U17.16 (VCC), U19.16 (VCC), U20.14 (VCC), R13.2, R14.2, R15.2, R16.2, R17.2, R18.2, R19.2, R20.2, R21.2, R22.2, R23.2, R24.2, R25.2
- net GND: now also U17.15 (~{EN}), U17.8 (GND), U19.15 (~{EN}), U19.8 (GND), U20.7 (GND), R26.2, SW3.1, SW3.2, SW3.3, SW3.4, SW3.5, SW3.6, SW3.7, SW3.8, SW4.1
- net clock_pulse: now also C8.2
- net at R12.1: now also D7.2 (A)
- net at U21.11 (I0d), U22.6 (Q3): now also R9.1, SW2.1, U21.10 (I1d)
- net at U18.11 (I0d): now also R21.1, SW3.9
- net at U18.12 (Qc): now also U14.12 (B6)
- net at U18.14 (I0c): now also R22.1, SW3.10
- net at U18.2 (I0a): now also R24.1, SW3.12
- net at U18.4 (Qa): now also U14.14 (B4)
- net at U18.5 (I0b): now also R23.1, SW3.11
- net at U18.7 (Qb): now also U14.13 (B5)
- net at U18.9 (Qd): now also U14.11 (B7)
- net at U17.1 (A/B): now also J2.NO, U19.1 (A/B), D7.1 (K)
- net at U17.11 (I0d): now also R20.1, SW3.13
- net at U17.12 (Qc): now also U14.16 (B2)
- net at U17.14 (I0c): now also R19.1, SW3.14
- net at U17.2 (I0a): now also R17.1, SW3.16
- net at U17.4 (Qa): now also U14.18 (B0)
- net at U17.5 (I0b): now also R18.1, SW3.15
- net at U17.7 (Qb): now also U14.17 (B1)
- net at U17.9 (Qd): now also U14.15 (B3)
- net at U20.1: now also C8.1, R26.1
- net control_logic: now reaches U20.2
- net at U20.3: now also U19.3 (I1a)
- net at J2.NC, U21.1 (A/B): now also D1.1 (K); no longer D1.2 (A)
- net at U15.8 (A2), U21.12 (Qc): now also D4.2 (A)
- net at U15.10 (A0), U21.4 (Qa): now also D6.2 (A)
- net at U15.9 (A1), U21.7 (Qb): now also D5.2 (A)
- net at U15.7 (A3), U21.9 (Qd): now also D3.2 (A)
- net at U14.19 (CE), U15.27 (~{WE}): now also U19.4 (Qa)
- net at R7.1: now also D1.2 (A); no longer D1.1 (K)
- new net: D6.1 (K), R16.1
- new net: D3.1 (K), R13.1
- new net: D5.1 (K), R15.1
- new net: R25.1, SW4.2
- new net: D4.1 (K), R14.1
Other:
- note added: "RAM"
- moved on the sheet: C3, C4, C5, C6, C7, J1B, J2B, R1, R10, R11, R12, R2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
