File: 8-Bit-Computer/8-Bit-Computer.kicad_sch (KiCad schematic)
At the start: 109 parts, among them IC1 AT28C64B-15SU-T, IC2 AT28C64B-15SU-T, IC3 AT28C64B-15SU-T, J1 XLR3_Switched, J2 XLR3_Switched, J3 XLR3_Switched, SW1 SW_Push, SW2 SW_DIP_x04, SW3 SW_DIP_x08, SW4 SW_Push, SW5 SW_Push, U1 NA555D, U10 74LS283, U11 74HC245, U12 74HC86, U13 74HC86, U14 74HC245, U15 HM62256BLP, U16 74HC245, U17 74157, U18 74157, U19 74157, U2 AMS1117-5.0, U20 74HC00, U21 74157, U22 HDSP-7403, U23 74LS377, U24 74LS377, U25 74LS377, U26 74HC245, U27 74LS161, U28 74HC245, U29 74LS377, U3 74HC00, U30 HDSP-7403, U31 74LS377, U32 HDSP-7403, U33 HDSP-7403, U34 74LS107, U35 NA555D, U36 74LS139, U37 74LS161, U38 74LS138, U39 74LS08, U4 LM555xM, U40 74LS04, U41 74LS04, U42 74LS377, U5 NA555D, U6 74HC00, U7 74HC245, U8 74LS02, U9 74LS283

Commit message: Completed Schematics Version 1
Parts:
- added C11, C12, C13, C14, C15, C16, C17, C18, C19, C20, C21, C22, C23, C24, C25, C26, C27, C28, C29, C30, C31, C32, C33, C34, C35, C36, C37, C38, C39, C40, C41, C42: C, symbol Device:C
- added D12, D13, D14, D15, D16, D17, D18, D19, D20, D21, D22, D23, D63, D64, D65, D66: B_LED, symbol Device:LED
- added D24, D25, D26, D27, D28, D29, D30, D31, D32, D33, D34, D35, D36, D37, D38, D39, D40, D41, D42, D43, D44, D45, D46, D47, D48, D49, D50, D51, D52, D53, D54, D55, D56, D57, D58, D59, D60, D61, D62, D80, D81, D82: R_LED, symbol Device:LED
- added D67, D68, D69, D70, D71, D72, D73, D74: Y_LED, symbol Device:LED
- added D75, D76, D77, D78, D79: G_LED, symbol Device:LED
- added R100, R101, R102, R103, R104, R105, R106, R107, R108, R109, R110, R111, R112, R113, R24, R32, R33, R34, R35, R40, R41, R42, R43, R44, R45, R46, R47, R48, R49, R50, R51, R52, R53, R54, R55, R56, R57, R58, R59, R60, R61, R62, R63, R64, R65, R66, R67, R68, R69, R70, R71, R72, R73, R74, R75, R76, R77, R78, R79, R80, R81, R82, R83, R84, R85, R86, R87, R88, R89, R90, R91, R92, R93, R94, R95, R96, R97, R98, R99: R_US, symbol Device:R_US
- added U43: 74LS00, symbol 74xx:74LS00
- added U44: 74HC00, symbol 74xx:74HC00
- D3: value G_LED -> R_LED
- D4, D5, D6: value G_LED -> B_LED
Connections:
- net #InstrReg_in is gone; now on net #II: U25.1 (~{E})
- net #InstrReg_out is gone; now on net #IO: U26.19 (CE)
- net #MEM_O is gone; now on net #RO: U16.19 (CE)
- net #PC_out is gone; now on net #CO: U28.19 (CE)
- net Addr_in is gone; now on net #MI: U31.1 (~{E})
- net SUB is gone; now on net SU: U12.1, U12.12, U12.4, U12.9, U13.1, U13.12, U13.4, U13.9, U9.7 (C0)
- net count_enable is gone; now on net CE: U27.10 (CET), U27.7 (CEP)
- net #CLR: now also U43.1, U43.10, U43.11, U43.9; no longer U20.11, U20.4, U20.5, U20.9
- net +5V: now also C11.1, C12.1, C13.1, C14.1, C15.1, C16.1, C17.1, C18.1, C19.1, C20.1, C21.1, C22.1, C23.1, C24.1, C25.1, C26.1, C27.1, C28.1, C29.1, C30.1, C31.1, C32.1, C33.1, C34.1, C35.1, C36.1, C37.1, C38.1, C39.1, C40.1, C41.1, C42.1, U43.14 (VCC); no longer R13.2, R14.2, R15.2, R16.2
- net AI: now also R14.1
- net ALU_0: now also R62.2
- net ALU_1: now also R63.2
- net ALU_2: now also R64.2
- net ALU_3: now also R65.2
- net ALU_4: now also R66.2
- net ALU_5: now also R67.2
- net ALU_6: now also R68.2
- net ALU_7: now also R69.2
- net AO: now also R24.1
- net BI: now also R44.1
- net BUS0: now also U26.14 (B4), R77.2, R78.1; no longer U26.18 (B0)
- net BUS1: now also U26.13 (B5), R76.2, R79.1; no longer U26.17 (B1)
- net BUS2: now also U26.12 (B6), R75.2, R80.1; no longer U26.16 (B2)
- net BUS3: now also U26.11 (B7), R74.2, R81.1; no longer U26.15 (B3)
- net BUS4: now also R73.2, R82.1; no longer U26.14 (B4)
- net BUS5: now also R72.2, R83.1; no longer U26.13 (B5)
- net BUS6: now also R71.2, R84.1; no longer U26.12 (B6)
- net BUS7: now also R70.2, R85.1; no longer U26.11 (B7)
- net CE: now also R42.1
- net CLR: now also U43.8; no longer U20.6
- net CL_IB1: now also R111.2
- net CL_IB2: now also R112.2
- net CL_IB3: now also R113.2
- net CO: now also R41.1
- net EO: now also R46.1
- net FI: now also R35.1
- net GND: now also D3.1 (K), D4.1 (K), D5.1 (K), D6.1 (K), C11.2, C12.2, C13.2, C14.2, C15.2, C16.2, C17.2, C18.2, C19.2, C20.2, C21.2, C22.2, C23.2, C24.2, C25.2, C26.2, C27.2, C28.2, C29.2, C30.2, C31.2, C32.2, C33.2, C34.2, C35.2, C36.2, C37.2, C38.2, C39.2, C40.2, C41.2, C42.2, D12.1 (K), D13.1 (K), D14.1 (K), D15.1 (K), D16.1 (K), D17.1 (K), D18.1 (K), D19.1 (K), D20.1 (K), D21.1 (K), D22.1 (K), D23.1 (K), D24.1 (K), D25.1 (K), D26.1 (K), D27.1 (K), D28.1 (K), D29.1 (K), D30.1 (K), D31.1 (K), D32.1 (K), D33.1 (K), D34.1 (K), D35.1 (K), D36.1 (K), D37.1 (K), D38.1 (K), D39.1 (K), D40.1 (K), D41.1 (K), D42.1 (K), D43.1 (K), D44.1 (K), D45.1 (K), D46.1 (K), D47.1 (K), D48.1 (K), D49.1 (K), D50.1 (K), D51.1 (K), D52.1 (K), D53.1 (K), D54.1 (K), D55.1 (K), D56.1 (K), D57.1 (K), D58.1 (K), D59.1 (K), D60.1 (K), D61.1 (K), D62.1 (K), D63.1 (K), D64.1 (K), D65.1 (K), D66.1 (K), D67.1 (K), D68.1 (K), D69.1 (K), D70.1 (K), D71.1 (K), D72.1 (K), D73.1 (K), D74.1 (K), D75.1 (K), D76.1 (K), D77.1 (K), D78.1 (K), D79.1 (K), D80.1 (K), D81.1 (K), D82.1 (K), R78.2, R79.2, R80.2, R81.2, R82.2, R83.2, R84.2, R85.2, U43.7 (GND)
- net HLT: now also R34.1
- net II: now also R15.1
- net IO: now also R16.1
- net IR_4: now also R94.1
- net IR_5: now also R95.1
- net IR_6: now also R96.1
- net IR_7: now also R97.1
- net J: now also R40.1
- net MI: now also R33.1
- net OI: now also U41.13, R43.1
- net RI: now also U14.19 (CE), R32.1, U44.10, U44.9
- net RO: now also R31.1
- net SU: now also R45.1
- net WRAM: no longer U14.19 (CE), U15.27 (~{WE})
- net clock_pulse: no longer R31.1, U23.11 (CP), U24.11 (CP), U25.11 (CP), U27.2 (CP), U29.11 (CP), U31.11 (CP), U37.2 (CP), U42.11 (CP), U6.8
- net B_3: now reaches U12.2, U24.9 (Q3)
- net B_3: now also R57.2
- net PC_2: now reaches R29.1, U27.13 (Q1), U28.3 (A1)
- net PC_1: now reaches R28.1, U27.12 (Q2), U28.4 (A2)
- net PC_0: now reaches R27.1, U27.11 (Q3), U28.5 (A3)
- net B_4: now reaches U13.2, U24.12 (Q4)
- net B_4: now also R58.2
- net A_4: now reaches U10.5 (A1), U23.12 (Q4), U7.6 (A4)
- net A_4: now also R50.2
- net A_5: now reaches U10.3 (A2), U23.15 (Q5), U7.7 (A5)
- net A_5: now also R51.2
- net A_6: now reaches U10.14 (A3), U23.16 (Q6), U7.8 (A6)
- net A_6: now also R52.2
- net A_7: now reaches U10.12 (A4), U23.19 (Q7), U7.9 (A7)
- net A_7: now also R53.2
- net A_0: now reaches U23.2 (Q0), U7.2 (A0), U9.5 (A1)
- net A_0: now also R13.2
- net A_1: now reaches U23.5 (Q1), U7.3 (A1), U9.3 (A2)
- net A_1: now also R47.2
- net A_2: now reaches U23.6 (Q2), U7.4 (A2), U9.14 (A3)
- net A_2: now also R48.2
- net A_3: now reaches U23.9 (Q3), U7.5 (A3), U9.12 (A4)
- net A_3: now also R49.2
- net IR_0: now reaches U25.2 (Q0), U26.6 (A4)
- net IR_0: now also R98.1
- net IR_1: now reaches U25.5 (Q1), U26.7 (A5)
- net IR_1: now also R99.1
- net IR_2: now reaches U25.6 (Q2), U26.8 (A6)
- net IR_2: now also R100.1
- net IR_3: now reaches U25.9 (Q3), U26.9 (A7)
- net IR_3: now also R101.1
- net B_0: now reaches U12.13, U24.2 (Q0)
- net B_0: now also R54.2
- net B_7: now reaches U13.13, U24.19 (Q7)
- net B_7: now also R61.2
- net MA_1: now reaches U15.9 (A1), U21.12 (Qc)
- net MA_1: now also R103.1; no longer D4.2 (A)
- net MA_3: now reaches U15.7 (A3), U21.4 (Qa)
- net MA_3: now also R105.1; no longer D5.2 (A)
- net MA_2: now reaches U15.8 (A2), U21.7 (Qb)
- net MA_2: now also R104.1; no longer D6.2 (A)
- net MA_0: now reaches U15.10 (A0), U21.9 (Qd)
- net MA_0: now also R102.1; no longer D3.2 (A)
- net at U38.10 (O5): now also U43.2; no longer U20.10
- net DEC_5: now reaches U38.11 (O4)
- net DEC_5: now also R110.1
- net DEC_4: now reaches U38.12 (O3)
- net DEC_4: now also R109.1
- net DEC_3: now reaches U38.13 (O2)
- net DEC_3: now also R108.1
- net DEC_2: now reaches U38.14 (O1)
- net DEC_2: now also R107.1
- net DEC_1: now reaches U38.15 (O0)
- net DEC_1: now also R106.1
- net #CLK: now reaches U6.10, U6.6, U6.9
- net #CLK: now also U37.2 (CP)
- net B_5: now reaches U13.5, U24.15 (Q5)
- net B_5: now also R59.2
- net B_6: now reaches U13.10, U24.16 (Q6)
- net B_6: now also R60.2
- net B_1: now reaches U12.10, U24.5 (Q1)
- net B_1: now also R55.2
- net B_2: now reaches U12.5, U24.6 (Q2)
- net B_2: now also R56.2
- net at R23.2, SW5.2: now also U43.12, U43.13; no longer U20.12, U20.13
- net at U37.1 (~{MR}): now also U43.6; no longer U41.12
- net at U20.8: no longer U41.13
- net MEM_0: now reaches U14.11 (B7), U15.19 (Q7), U16.9 (A7)
- net MEM_0: now also R86.2
- net MEM_1: now reaches U14.12 (B6), U15.18 (Q6), U16.8 (A6)
- net MEM_1: now also R87.2
- net MEM_2: now reaches U14.13 (B5), U15.17 (Q5), U16.7 (A5)
- net MEM_2: now also R88.2
- net MEM_3: now reaches U14.14 (B4), U15.16 (Q4), U16.6 (A4)
- net MEM_3: now also R89.2
- net MEM_4: now reaches U14.15 (B3), U15.15 (Q3), U16.5 (A3)
- net MEM_4: now also R90.2
- net MEM_5: now reaches U14.16 (B2), U15.13 (Q2), U16.4 (A2)
- net MEM_5: now also R91.2
- net MEM_6: now reaches U14.17 (B1), U15.12 (Q1), U16.3 (A1)
- net MEM_6: now also R92.2
- net MEM_7: now reaches U14.18 (B0), U15.11 (Q0), U16.2 (A0)
- net MEM_7: now also R93.2
- net at D11.2 (A): now also R24.2; no longer R31.2
- net at R13.1: now also D3.2 (A); no longer D3.1 (K)
- net LSB renamed PC_3
- net Res_load_enable renamed #OI
- net #OI: now also U41.12
- new net: D80.2 (A), R111.1
- new net: D37.2 (A), R60.1
- new net: D68.2 (A), R99.2
- new net: D32.2 (A), R55.1
- new net: D23.2 (A), R46.2
- new net: U43.3, U43.4, U43.5
- new net: D46.2 (A), R69.1
- new net: D33.2 (A), R56.1
- new net: D29.2 (A), R52.1
- new net: D78.2 (A), R109.2
- new net: D64.2 (A), R95.2
- new net: D70.2 (A), R101.2
- new net: D72.2 (A), R103.2
- new net: D54.2 (A), R77.1
- new net: D20.2 (A), R43.2
- new net: D38.2 (A), R61.1
- new net: D17.2 (A), R40.2
- new net: D44.2 (A), R67.1
- new net: D53.2 (A), R76.1
- new net: D13.2 (A), R32.2
- new net: D79.2 (A), R110.2
- new net: D82.2 (A), R113.1
- new net: D75.2 (A), R106.2
- new net: D56.2 (A), R87.1
- new net: U15.27 (~{WE}), U44.8
- new net: D47.2 (A), R70.1
- new net: D57.2 (A), R88.1
- new net: D31.2 (A), R54.1
- new net: D5.2 (A), R15.2
- new net: D58.2 (A), R89.1
- new net: D6.2 (A), R16.2
- new net: D39.2 (A), R62.1
- new net: D18.2 (A), R41.2
- new net: D35.2 (A), R58.1
- new net: D63.2 (A), R94.2
- new net: D71.2 (A), R102.2
- new net: D51.2 (A), R74.1
- new net: D60.2 (A), R91.1
- new net: D15.2 (A), R34.2
- new net: D16.2 (A), R35.2
- new net: D22.2 (A), R45.2
- new net: D34.2 (A), R57.1
- new net: D30.2 (A), R53.1
- new net: D73.2 (A), R104.2
- new net: D14.2 (A), R33.2
- new net: D21.2 (A), R44.2
- new net: D66.2 (A), R97.2
- new net: D25.2 (A), R48.1
- new net: D81.2 (A), R112.1
- new net: D61.2 (A), R92.1
- new net: D19.2 (A), R42.2
- new net: D74.2 (A), R105.2
- new net: D36.2 (A), R59.1
- new net: D65.2 (A), R96.2
- new net: D27.2 (A), R50.1
- new net: D67.2 (A), R98.2
- new net: D76.2 (A), R107.2
- new net: D77.2 (A), R108.2
- new net: D4.2 (A), R14.2
- new net: D28.2 (A), R51.1
- new net: D42.2 (A), R65.1
- new net: D43.2 (A), R66.1
- new net: D62.2 (A), R93.1
- new net: D41.2 (A), R64.1
- new net: D45.2 (A), R68.1
- new net: D48.2 (A), R71.1
- new net: D52.2 (A), R75.1
- new net: D40.2 (A), R63.1
- new net: D26.2 (A), R49.1
- new net: D24.2 (A), R47.1
- new net: D59.2 (A), R90.1
- new net: D55.2 (A), R86.1
- new net: D49.2 (A), R72.1
- new net: D12.2 (A), R31.2
- new net: D50.2 (A), R73.1
- new net: D69.2 (A), R100.2
- new net CLK: U23.11 (CP), U24.11 (CP), U25.11 (CP), U27.2 (CP), U29.11 (CP), U31.11 (CP), U42.11 (CP), U6.8
- no-connect marks 1 -> 2
