File: 8-Bit-Computer/8-Bit-Computer.kicad_pcb (KiCad board)
At the start: 2 copper layers, 293 parts, among them IC1 AT28C64B-15SU-T, IC2 AT28C64B-15SU-T, IC3 AT28C64B-15SU-T, SW1 SW_Push, SW2 SW_DIP_x04, SW3 SW_DIP_x08, SW4 SW_Push, SW5 SW_Push, SW6 SW_Push_DPDT, SW7 SW_Push_DPDT, SW8 SW_Push_DPDT, U1 NA555D, U10 74LS283, U11 74HC245, U12 74HC86, U13 74HC86, U14 74HC245, U15 HM62256BLP, U16 74HC245, U17 74157, U18 74157, U19 74157, U2 AMS1117-5.0, U20 74HC00, U21 74157, U22 HDSP-7403, U23 74LS377, U24 74LS377, U25 74LS377, U26 74HC245, U27 74LS161, U28 74HC245, U29 74LS377, U3 74HC00, U30 HDSP-7403, U31 74LS377, U32 HDSP-7403, U33 HDSP-7403, U34 74LS107, U35 NA555D, U36 74LS139, U37 74LS161, U38 74LS138, U39 74LS08, U4 NA555D, U40 74LS04, U41 74LS04, U42 74LS377, U43 74LS00, U44 74HC00, U5 NA555D, U6 74HC00, U7 74HC245, U8 74LS02, U9 74LS283

Commit message: finished the PCB layout for ALU and clock
Parts:
- added SW9: SW_Push_Dual, Button_Switch_THT:SW_PUSH_6mm, F.Cu at (198.0, 122.0)
- C18, C19, C22, C23, U11, U23: moved to B.Cu
- SW6, SW7, SW8: footprint Button_Switch_THT:SW_Tactile_SKHH_Angled -> Button_Switch_THT:SW_Push_2P2T_Toggle_CK_PVA2xxH4xxxxxxV2
- moved D3 385.4 mm to (417.0, 200.5), turned to 180 degrees
- moved D25 377.4 mm to (417.0, 196.5), turned to 180 degrees
- moved D26 376.1 mm to (417.0, 194.5), turned to 180 degrees
- moved D31 376.0 mm to (427.4, 147.5), turned to 180 degrees
- moved D32 375.9 mm to (427.4, 149.5), turned to 180 degrees
- moved D33 375.8 mm to (427.4, 151.5), turned to 180 degrees
- moved D34 375.7 mm to (427.4, 153.5), turned to 180 degrees
- moved D35 375.6 mm to (427.4, 155.5), turned to 180 degrees
- moved D36 375.5 mm to (427.4, 157.5), turned to 180 degrees
- moved D37 375.3 mm to (427.4, 159.5), turned to 180 degrees
- moved D38 375.1 mm to (427.4, 161.5), turned to 180 degrees
- moved D27 374.9 mm to (417.0, 192.5), turned to 180 degrees
- moved D24 374.8 mm to (417.0, 198.5), turned to 180 degrees
- moved D28 373.7 mm to (417.0, 190.5), turned to 180 degrees
- moved D29 372.6 mm to (417.0, 188.5), turned to 180 degrees
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Connections:
- RV1 pad 1: Net-(U1-THR) -> unconnected-(RV1-Pad1)
- RV1 pad 3: unconnected-(RV1-Pad3) -> Net-(U1-THR)
- U20 pad 4: unconnected-(U20-Pad4) -> /RI
- U20 pad 5: unconnected-(U20-Pad5) -> /RI
- U20 pad 6: unconnected-(U20-Pad6) -> Net-(U15-~{WE})
Routing:
- net /BUS0: track 0.00 -> 158.1 mm, vias 0 -> 6
- net /BUS1: track 0.00 -> 150.8 mm, vias 0 -> 6
- net /BUS2: track 0.00 -> 142.3 mm, vias 0 -> 6
- net /BUS3: track 0.00 -> 135.3 mm, vias 0 -> 6
- net /BUS4: track 0.00 -> 133.3 mm, vias 0 -> 5
- net /BUS5: track 0.00 -> 129.9 mm, vias 0 -> 5
- net /BUS6: track 0.00 -> 128.7 mm, vias 0 -> 5
- net /BUS7: track 0.00 -> 125.0 mm, vias 0 -> 5
- net /SU: track 0.00 -> 114.3 mm, vias 0 -> 12
- net GND: track 0.00 -> 114.0 mm, vias 0 -> 31
- net /CLK: track 0.00 -> 90.1 mm, vias 0 -> 3
- net /#AO: track 0.00 -> 77.5 mm, vias 0 -> 3
- net Net-(U10-C4): track 0.00 -> 70.4 mm, vias 0 -> 3
- net /ALU_7: track 0.00 -> 69.7 mm, vias 0 -> 5
- net /ALU_6: track 0.00 -> 66.3 mm, vias 0 -> 7
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Other:
- copper layers 2 -> 4
- board text added: "Clock Speed"
- board text added: "Debouncers"
- board text added: "Manual Clock"
- board text added: "Oscillator"
- board text added: "Toggle Manual"

Commit message: completed display
Parts:
- removed U33: HDSP-7403, Display_7Segment:HDSP-7401
- added D83: B_LED, LED_SMD:LED_0805_2012Metric, F.Cu at (32.9, -25.5)
- added R114: R_US, Resistor_SMD:R_0402_1005Metric, F.Cu at (30.5, -26.5)
- added U44: D1X8K-14BL, Display_7Segment:D1X8K, F.Cu at (33.1, 162.9)
- C10, C29, C30, C9, R21, R22, U29, U35: moved to B.Cu
- U22, U30, U32: value HDSP-7403 -> D1X8K-14BL; footprint Display_7Segment:HDSP-7401 -> Display_7Segment:D1X8K
- moved U37 426.7 mm to (511.6, -8.55)
- moved U40 426.7 mm to (508.9, 23.2)
- moved U43 426.7 mm to (500.5, 33.5)
- moved U38 426.7 mm to (520.0, -8.55)
- moved U41 426.7 mm to (492.0, 33.5)
- moved IC2 387.6 mm to (447.0, -18.0)
- moved IC3 387.6 mm to (466.4, -18.0)
- moved C11 377.3 mm to (37.0, -42.4)
- moved C12 377.3 mm to (37.5, -34.4)
- moved C13 377.3 mm to (37.0, -27.4)
- moved C14 377.3 mm to (30.0, -37.9)
- moved C15 377.3 mm to (30.5, -49.9)
- moved C3 377.3 mm to (43.0, -42.9)
- moved C4 377.3 mm to (44.0, -44.9)
- moved C5 377.3 mm to (44.1, -38.0)
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Connections:
- IC1 pad 15: /LCD_B -> /LCD_D
- U22 pad 1: Net-(U36A-O0) -> /LCD_E
- U22 pad 10: /LCD_A -> /LCD_G
- U22 pad 2: /LCD_F -> /LCD_D
- U22 pad 3: /LCD_G -> Net-(U36A-O1)
- U22 pad 4: /LCD_E -> /LCD_C
- U22 pad 5: /LCD_B -> GND
- U22 pad 6: Net-(U36A-O0) -> /LCD_B
- U22 pad 7: GND -> /LCD_A
- U22 pad 8: /LCD_C -> Net-(U36A-O1)
- U22 pad 9: /LCD_B -> /LCD_F
- U30 pad 1: Net-(U36A-O1) -> /LCD_E
- U30 pad 10: /LCD_A -> /LCD_G
- U30 pad 2: /LCD_F -> /LCD_D
- U30 pad 3: /LCD_G -> Net-(U36A-O2)
- U30 pad 4: /LCD_E -> /LCD_C
- U30 pad 5: /LCD_B -> GND
- U30 pad 6: Net-(U36A-O1) -> /LCD_B
- U30 pad 7: GND -> /LCD_A
- U30 pad 8: /LCD_C -> Net-(U36A-O2)
- U30 pad 9: /LCD_B -> /LCD_F
- U32 pad 1: Net-(U36A-O2) -> /LCD_E
- U32 pad 10: /LCD_A -> /LCD_G
- U32 pad 2: /LCD_F -> /LCD_D
- U32 pad 3: /LCD_G -> Net-(U36A-O3)
- U32 pad 4: /LCD_E -> /LCD_C
- U32 pad 5: /LCD_B -> GND
- U32 pad 6: Net-(U36A-O2) -> /LCD_B
- U32 pad 7: GND -> /LCD_A
- U32 pad 8: /LCD_C -> Net-(U36A-O3)
- U32 pad 9: /LCD_B -> /LCD_F
Routing:
- net /LCD_E: track 0.00 -> 147.2 mm, vias 0 -> 5
- net /LCD_C: track 0.00 -> 138.3 mm, vias 0 -> 4
- net /LCD_D: track 0.00 -> 135.0 mm, vias 0 -> 4
- net /LCD_F: track 0.00 -> 80.8 mm, vias 0 -> 5
- net /LCD_A: track 0.00 -> 80.0 mm, vias 0 -> 5
- net /LCD_G: track 0.00 -> 77.9 mm, vias 0 -> 4
- net /LCD_B: track 0.00 -> 77.1 mm, vias 0 -> 4
- net Net-(U36A-O3): track 0.00 -> 67.1 mm, vias 0 -> 2
- net Net-(IC1-A8): track 0.00 -> 66.6 mm, vias 0 -> 6
- net Net-(U36A-O2): track 0.00 -> 53.2 mm, vias 0 -> 2
- net Net-(IC1-A9): track 0.00 -> 46.1 mm, vias 0 -> 2
- net /#OI: track 0.00 -> 45.4 mm, vias 0 -> 3
- net Net-(IC1-A10): track 0.00 -> 45.4 mm, vias 0 -> 2
- net /CLK: track 90.1 -> 133.9 mm, vias 3 -> 6
- net /BUS7: track 125.0 -> 166.6 mm, vias 5 -> 7
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Other:
- board outline added: 150 x 150 mm

Commit message: Finished Ram and started control logic
Parts:
- removed the U44 at (191.0, -59.5)
- R10, R11, R17, R18, R19, R20, R25, R36, R37, R38, R39, R8, R9, U20, U21, U40, U41: moved to B.Cu
- moved U18 326.9 mm to (85.9, 102.4), turned to 90 degrees
- moved U17 324.8 mm to (75.4, 102.4), turned to 90 degrees
- moved C8 317.6 mm to (71.5, 70.0)
- moved U19 310.0 mm to (74.4, 61.0), turned to 90 degrees
- moved U14 309.0 mm to (87.4, 80.5), turned to 90 degrees
- moved U20 308.6 mm to (74.5, 69.5), turned to -90 degrees
- moved U21 288.5 mm to (64.4, 102.4), turned to -90 degrees
- moved U31 277.5 mm to (53.9, 102.4), turned to -90 degrees
- moved U16 276.6 mm to (71.9, 80.5), turned to -90 degrees
- moved U15 266.9 mm to (46.4, 52.6)
- moved SW3 264.1 mm to (83.1, 112.6), turned to 90 degrees
- moved SW2 260.9 mm to (72.8, 112.4), turned to 90 degrees
- moved R38 254.7 mm to (87.4, 109.4), turned to -90 degrees
- moved R37 253.5 mm to (86.4, 109.4), turned to -90 degrees
- moved R19 253.4 mm to (83.9, 109.4), turned to -90 degrees
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Routing:
- net Net-(U19-I0a): track 0.00 -> 114.3 mm, vias 0 -> 4
- net /#MI: track 0.00 -> 107.6 mm, vias 0 -> 4
- net GND: track 136.6 -> 219.1 mm, vias 42 -> 64
- net /SU: track 114.8 -> 196.4 mm, vias 12 -> 13
- net /BUS3: track 154.2 -> 231.4 mm, vias 6 -> 9
- net /BUS6: track 165.1 -> 240.3 mm, vias 7 -> 10
- net /#OI: track 45.4 -> 119.7 mm
- net /BUS2: track 160.5 -> 232.5 mm, vias 6 -> 9
- net /BUS1: track 167.7 -> 238.7 mm, vias 6 -> 11
- net /BUS0: track 174.3 -> 239.5 mm, vias 6 -> 9
- net /MEM_7: track 0.00 -> 64.7 mm, vias 0 -> 4
- net /MEM_6: track 0.00 -> 60.2 mm, vias 0 -> 3
- net /CLK: track 133.9 -> 190.9 mm, vias 6 -> 8
- net /EO: track 0.00 -> 55.4 mm, vias 0 -> 3
- net /MA_1: track 0.00 -> 54.6 mm, vias 0 -> 4
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Other:
- board size 150 x 150 mm -> 145 x 131 mm

Commit message: remaining to fit in clock
Parts:
- R23, U27, U37, U38, U43: moved to B.Cu
- moved U38 261.2 mm to (154.8, 66.7), turned to 180 degrees
- moved R23 254.8 mm to (169.0, 78.7)
- moved U37 251.2 mm to (155.0, 78.2), turned to 180 degrees
- moved U43 226.6 mm to (153.8, 90.2), turned to 180 degrees
- moved SW5 203.2 mm to (166.2, 81.9), turned to 90 degrees
- moved IC2 200.8 mm to (128.0, 61.7)
- moved U40 200.8 mm to (135.6, 75.7)
- moved U41 200.8 mm to (135.6, 86.7)
- moved IC3 200.8 mm to (147.4, 61.7)
- moved U25 152.6 mm to (87.0, 70.0), turned to -90 degrees
- moved U26 151.6 mm to (90.0, 58.5), turned to -90 degrees
- moved U28 146.8 mm to (136.3, 52.8), turned to 90 degrees
- moved U27 140.5 mm to (134.6, 51.5), turned to -90 degrees
- moved C15 128.1 mm to (39.8, 96.9)
- moved U3 128.1 mm to (37.3, 102.0)
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Routing:
- net /BUS3: track 231.4 -> 358.4 mm, vias 9 -> 14
- net /BUS2: track 232.5 -> 355.8 mm, vias 9 -> 14
- net /BUS1: track 238.7 -> 359.5 mm, vias 11 -> 16
- net /BUS0: track 239.5 -> 356.3 mm, vias 9 -> 14
- net /BUS5: track 210.9 -> 282.4 mm, vias 11 -> 14
- net /#CO: track 15.2 -> 81.4 mm, vias 2 -> 5
- net /RI: track 36.9 -> 102.6 mm, vias 1 -> 5
- net /BUS4: track 211.0 -> 272.0 mm, vias 11 -> 14
- net /CF: track 74.2 -> 132.7 mm
- net /#RO: track 37.6 -> 94.5 mm, vias 2 -> 5
- net /#J: track 16.5 -> 73.2 mm, vias 2 -> 4
- net /ZF: track 91.8 -> 147.9 mm
- net /#IO: track 1.55 -> 54.8 mm, vias 1 -> 3
- net /IR_4: track 35.8 -> 88.6 mm, vias 2 -> 7
- net /#AI: track 76.4 -> 118.6 mm
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
Commit message: need to place leds
Parts:
- removed SW9: SW_Push_Dual, Button_Switch_THT:SW_PUSH_6mm
- U3: moved to B.Cu
- moved D61 308.1 mm to (18.3, 7.17)
- moved D62 308.1 mm to (18.3, 10.2)
- moved D55 303.0 mm to (17.1, 17.8)
- moved D56 303.0 mm to (17.1, 20.9)
- moved D57 303.0 mm to (17.1, 23.9)
- moved D58 303.0 mm to (17.1, 27.0)
- moved D59 303.0 mm to (17.1, 30.0)
- moved D60 303.0 mm to (17.1, 33.0)
- moved R92 281.8 mm to (9.49, 14.5)
- moved R93 281.8 mm to (9.49, 16.5)
- moved D73 280.1 mm to (58.0, 23.6)
- moved D74 280.1 mm to (58.0, 26.6)
- moved R86 276.9 mm to (9.76, 20.9)
- moved R87 276.9 mm to (9.76, 22.9)
- moved R88 276.9 mm to (9.76, 24.9)
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Routing:
- net /IR_5: track 67.4 -> 112.9 mm, vias 5 -> 7
- net Net-(D66-A): track 0.00 -> 45.3 mm, vias 0 -> 4
- net /IR_6: track 67.6 -> 108.1 mm, vias 3 -> 5
- net Net-(D65-A): track 0.00 -> 36.4 mm, vias 0 -> 4
- net Net-(U3-Pad3): track 11.5 -> 47.7 mm, vias 0 -> 3
- net /IR_4: track 88.6 -> 123.9 mm, vias 7 -> 10
- net /IR_7: track 64.3 -> 99.3 mm, vias 4 -> 6
- net Net-(U3-Pad6): track 9.50 -> 43.8 mm, vias 0 -> 3
- net Net-(D64-A): track 0.00 -> 28.1 mm, vias 0 -> 4
- net Net-(U3-Pad11): track 21.1 -> 49.1 mm, vias 2 -> 1
- net Net-(D63-A): track 0.00 -> 20.2 mm, vias 0 -> 2
- net Net-(U5-Q): track 30.0 -> 47.5 mm, vias 2 -> 5
- net /PROG: track 44.2 -> 61.1 mm, vias 5 -> 6
- net /ZF: track 147.9 -> 164.7 mm, vias 3 -> 6
- net Net-(D70-A): track 0.00 -> 15.9 mm
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
Commit message: done with all LEDs except control word
Parts:
- moved C2 274.3 mm to (167.5, 126.5)
- moved C1 273.8 mm to (160.7, 133.5)
- moved U2 273.8 mm to (167.5, 133.0)
- moved D83 254.6 mm to (79.8, -28.6)
- moved R114 254.6 mm to (80.8, -31.0)
- moved R93 78.3 mm to (78.0, 54.5), turned to -90 degrees
- moved R92 77.6 mm to (76.0, 54.5), turned to -90 degrees
- moved R91 68.5 mm to (74.0, 54.5), turned to -90 degrees
- moved R90 67.3 mm to (72.0, 54.5), turned to -90 degrees
- moved D62 66.5 mm to (74.0, 46.5), turned to -90 degrees
- moved R89 66.3 mm to (70.0, 54.5), turned to -90 degrees
- moved D61 65.7 mm to (71.0, 46.5), turned to -90 degrees
- moved R88 65.3 mm to (68.0, 54.5), turned to -90 degrees
- moved R87 64.5 mm to (66.0, 54.5), turned to -90 degrees
- moved R86 63.4 mm to (63.5, 54.5), turned to -90 degrees
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Routing:
- net /BUS4: track 272.0 -> 351.3 mm, vias 14 -> 17
- net /BUS7: track 253.2 -> 313.3 mm, vias 11 -> 13
- net /BUS6: track 278.5 -> 335.9 mm, vias 12 -> 16
- net /DEC_4: track 0.00 -> 50.8 mm, vias 0 -> 7
- net /PC_3: track 7.80 -> 53.5 mm, vias 1 -> 6
- net /BUS5: track 282.4 -> 327.6 mm, vias 14 -> 18
- net /MEM_6: track 60.2 -> 103.1 mm, vias 3 -> 7
- net /MA_0: track 52.2 -> 93.5 mm, vias 4 -> 6
- net /MEM_7: track 64.7 -> 104.6 mm, vias 4 -> 8
- net GND: track 245.5 -> 278.6 mm, vias 74 -> 77
- net /MEM_5: track 52.6 -> 84.5 mm
- net /MEM_4: track 40.8 -> 71.6 mm, vias 3 -> 5
- net /DEC_2: track 0.00 -> 30.6 mm, vias 0 -> 5
- net /DEC_3: track 0.00 -> 28.8 mm, vias 0 -> 5
- net /MEM_3: track 39.3 -> 68.1 mm
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
Commit message: fixing errors
Routing:
- net GND: track 278.6 -> 378.4 mm, vias 77 -> 89
- net /HLT: track 34.5 -> 129.2 mm, vias 1 -> 3
- net +5V: track 154.6 -> 160.4 mm, vias 46 -> 48
- net /B_1: track 54.3 -> 50.9 mm
- net Net-(IC1-A7): track 4.95 -> 6.36 mm
- net /SU: track 196.0 -> 197.0 mm
- net /BUS7: track 313.3 -> 314.1 mm
- net /B_5: track 46.6 -> 47.3 mm
- net /IO: track 37.2 -> 37.9 mm
- net /A_7: vias 6 -> 4
