File: 8-Bit-Computer/8-Bit-Computer.kicad_pcb (KiCad board)
At the start: 4 copper layers, 145 x 131 mm, 294 parts, among them IC1 AT28C64B-15SU-T, IC2 AT28C64B-15SU-T, IC3 AT28C64B-15SU-T, SW1 SW_Push, SW2 SW_DIP_x04, SW3 SW_DIP_x08, SW4 SW_Push, SW5 SW_Push, SW6 SW_Push_DPDT, SW7 SW_Push_DPDT, SW8 SW_Push_DPDT, U1 NA555D, U10 74LS283, U11 74HC245, U12 74HC86, U13 74HC86, U14 74HC245, U15 HM62256BLP, U16 74HC245, U17 74157, U18 74157, U19 74157, U2 AMS1117-5.0, U20 74HC00, U21 74157, U22 D1X8K-14BL, U23 74LS377, U24 74LS377, U25 74LS377, U26 74HC245, U27 74LS161, U28 74HC245, U29 74LS377, U3 74HC00, U30 D1X8K-14BL, U31 74LS377, U32 D1X8K-14BL, U34 74LS107, U35 NA555D, U36 74LS139, U37 74LS161, U38 74LS138, U39 74LS08, U4 NA555D, U40 74LS04, U41 74LS04, U42 74LS377, U43 74LS00, U44 D1X8K-14BL, U5 NA555D, U6 74HC00, U7 74HC245, U8 74LS02, U9 74LS283

Commit message: removed control word LEDs
Parts:
- removed D11, D12, D13, D14, D15, D16, D17, D18, D19, D20, D21, D22, D23, D4, D5, D6, D83: B_LED, LED_SMD:LED_0805_2012Metric
- removed R114, R14, R15, R16, R24, R31, R32, R33, R34, R35, R40, R41, R42, R43, R44, R45, R46: R_US, Resistor_SMD:R_0402_1005Metric
- C32, C34, C35, C37, C38, C41: moved to B.Cu
- moved C40 278.7 mm to (60.5, 105.5)
- moved C41 278.3 mm to (58.0, 105.0), turned to 90 degrees
- moved C39 267.5 mm to (71.0, 97.5)
- moved C42 255.8 mm to (82.0, 97.0), turned to 90 degrees
- moved C32 250.8 mm to (64.0, 76.5), turned to -90 degrees
- moved C33 245.6 mm to (79.5, 84.5), turned to 180 degrees
- moved C37 237.5 mm to (68.0, 72.0), turned to 180 degrees
- moved C34 234.6 mm to (59.0, 53.0), turned to 180 degrees
- moved C38 210.6 mm to (94.5, 61.5), turned to 180 degrees
- moved C35 188.2 mm to (145.5, 62.5), turned to -90 degrees
- moved C36 177.7 mm to (166.0, 62.0)
Routing:
- net GND: track 378.4 -> 400.8 mm, vias 89 -> 94
- net +5V: track 160.4 -> 180.9 mm, vias 48 -> 51
- net /HLT: track 129.2 -> 130.4 mm
- net /MEM_0: track 59.7 -> 60.8 mm
- net /BUS3: track 376.7 -> 377.7 mm
- net /BUS5: track 327.6 -> 326.7 mm
Other:
- rule pad_to_mask_clearance: 0 -> 0.038
